File: Fan-Carrier.kicad_pcb (KiCad board)
At the start: 2 copper layers, 90 x 32 mm, 21 parts, among them J1 TC2030, J2 RJHSE-5381, M1 Fan_4pin, U1 AZ1117-3.3, U2 P3T1750DP

Commit message: finished PCB artwork
Routing:
- net GND: vias 0 -> 25
- net Earth: vias 0 -> 11

Commit message: increased thermal relief updated holddown nut solder paste pattern
Parts:
- J3: footprint openPoENode:119A-80A00-R02 -> openPoeNode:119A-80A00-R02
- J4: footprint openPoENode:119A-NUT-80-R02 -> openPoeNode:119A-NUT-80-R02
- U2: value P3T1750DP -> LM75

Commit message: prettification
Parts:
- added G***: LOGO, LOGO, B.Cu at (65.0, -16.0)
Other:
- board text added: "REV ${REVISION}"
